File: Hardware/C64/Xlink_CR.kicad_pcb (KiCad board)
At the start: 2 copper layers, 50 x 40 mm, 22 parts, among them J1 Prog, J2 Serial, J3 Prog, J4 C128-Reset, J5 Reset, P1 USB_Micro, P2 C64_Userport, U1 CH552T

Commit message: Updated C64-PCB, added pictures
Other:
- net class Default removed
- board text added: "Design 2022 by Thomas Tahsin-Bey"
- board text removed: "Design 2021 by Thomas Tahsin-Bey"
