File: Hardware/C64/Xlink_CR.kicad_sch (KiCad schematic)
At the start: 22 parts

Commit message: Updated C64-PCB, added pictures
Parts:
- C1: value (none) -> 4,7nF; footprint (none) -> TTB_MyLib:TTB_C0603
- C2, C3: value (none) -> 100nF; footprint (none) -> TTB_MyLib:TTB_C0603
- D1: value (none) -> CD4148WTP; footprint (none) -> TTB_MyLib:TTB_D0603
- J1: value (none) -> Prog; footprint (none) -> TTB_MyLib:TTB_Pinhead_2x1_2mm
- J2: value (none) -> Serial; footprint (none) -> TTB_MyLib:TTB_Pinhead_1x3_Rahmen
- J3: value (none) -> Prog; footprint (none) -> TTB_MyLib:TTB_Pinhead_1x2_Rahmen
- J4: value (none) -> C128-Reset; footprint (none) -> TTB_MyLib:TTB_Pinhead_1x1_Rahmen
- J5: value (none) -> Reset; footprint (none) -> Measurement_Points:Measurement_Point_Round-SMD-Pad_Small
- JP1: value (none) -> Cut for C128-Reset; footprint (none) -> Jumper:SolderJumper-2_P1.3mm_Bridged_Pad1.0x1.5mm
- MH1, MH2, MH3: value (none) -> Hole; footprint (none) -> Mounting_Holes:MountingHole_3mm
- P1: value (none) -> USB_Micro; footprint (none) -> TTB_MyLib:TTB_USB-B_Micro_LCSC_C10418
- P2: value (none) -> C64_Userport; footprint (none) -> TTB_MyLib:TTB_C64_Userport
- R1: value (none) -> 1M; footprint (none) -> TTB_MyLib:TTB_R0603
- R2: value (none) -> 20k; footprint (none) -> TTB_MyLib:TTB_R0603
- R3: value (none) -> 180R; footprint (none) -> TTB_MyLib:TTB_R0603
- RP1, RP2: value (none) -> 470R; footprint (none) -> TTB_MyLib:TTB_RNet1206_4R
- RP3: value (none) -> 1k0; footprint (none) -> TTB_MyLib:TTB_RNet1206_2R
- U1: value (none) -> CH552T; footprint (none) -> Housings_SSOP:TSSOP-20_4.4x6.5mm_Pitch0.65mm
